Commit message: Added Tiago description

File: pycram/resources/robots/tiago_dual.urdf (robot description, URDF)
Before this commit: robot tiago_dual, 69 links, 68 joints
Links:
- link arm_left_1_link: geometry collision mesh filename=package://iai_tiago_description/meshes/arm/arm_1_collision.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 scale=1 -1 -1; visual mesh filename=package://iai_tiago_description/meshes/arm/arm_1.stl scale=1 -1 -1
- link arm_left_2_link: geometry collision mesh filename=package://iai_tiago_description/meshes/arm/arm_2_collision.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 scale=1 1 -1; visual mesh filename=package://iai_tiago_description/meshes/arm/arm_2.stl scale=1 1 -1
- link arm_left_3_link: geometry collision mesh filename=package://iai_tiago_description/meshes/arm/arm_3_collision.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 scale=1 1 -1; visual mesh filename=package://iai_tiago_description/meshes/arm/arm_3.stl scale=1 1 -1
- link arm_left_4_link: geometry collision mesh filename=package://iai_tiago_description/meshes/arm/arm_4_collision.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 scale=-1 -1 -1; visual mesh filename=package://iai_tiago_description/meshes/arm/arm_4.stl scale=-1 -1 -1
- link arm_left_5_link: geometry collision mesh filename=package://iai_tiago_description/meshes/arm/arm_5_collision-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 scale=-1 -1 -1; visual mesh filename=package://iai_tiago_description/meshes/arm/arm_5-wrist-2017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 scale=-1 -1 -1
- link arm_left_6_link: geometry collision mesh filename=package://iai_tiago_description/meshes/arm/arm_6_collision-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 scale=-1 1 1; visual mesh filename=package://iai_tiago_description/meshes/arm/arm_6-wrist-2017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 scale=-1 1 1
- link arm_right_1_link: geometry collision mesh filename=package://iai_tiago_description/meshes/arm/arm_1_collision.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 scale=1 -1 1; visual mesh filename=package://iai_tiago_description/meshes/arm/arm_1.stl scale=1 -1 1
- link arm_right_2_link: geometry collision mesh filename=package://iai_tiago_description/meshes/arm/arm_2_collision.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 scale=1 1 1; visual mesh filename=package://iai_tiago_description/meshes/arm/arm_2.stl scale=1 1 1
- link arm_right_3_link: geometry collision mesh filename=package://iai_tiago_description/meshes/arm/arm_3_collision.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 scale=1 1 1; visual mesh filename=package://iai_tiago_description/meshes/arm/arm_3.stl scale=1 1 1
- link arm_right_4_link: geometry collision mesh filename=package://iai_tiago_description/meshes/arm/arm_4_collision.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 scale=1 1 1; visual mesh filename=package://iai_tiago_description/meshes/arm/arm_4.stl scale=1 1 1
- link arm_right_5_link: geometry collision mesh filename=package://iai_tiago_description/meshes/arm/arm_5_collision-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 scale=1 1 1; visual mesh filename=package://iai_tiago_description/meshes/arm/arm_5-wrist-2017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 scale=1 1 1
- link arm_right_6_link: geometry collision mesh filename=package://iai_tiago_description/meshes/arm/arm_6_collision-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 scale=1 1 1; visual mesh filename=package://iai_tiago_description/meshes/arm/arm_6-wrist-2017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 scale=1 1 1
- link head_1_link: geometry collision mesh filename=package://iai_tiago_description/meshes/head/head_1_collisio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 scale=1 1 1; visual mesh filename=package://iai_tiago_description/meshes/head/head_1.stl scale=1 1 1
- link head_2_link: geometry collision mesh filename=package://iai_tiago_description/meshes/head/head_2_collisio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 scale=1 1 1; visual mesh filename=package://iai_tiago_description/meshes/head/head_2.stl scale=1 1 1
- link torso_fixed_link: geometry collision box size=0.25 0.25 0.1; collision box size=0.4 0.25 0.04
- link torso_lift_link: geometry collision mesh filename=package://iai_tiago_description/meshes/torso/torso_lift_col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 scale=1 1 1; collision mesh filename=package://iai_tiago_description/meshes/torso/torso_lift_col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 scale=1 1 1
