Commit message: final excellence demo state

File: pycram/resources/robots/stretch_description.urdf (robot description, URDF)
Before this commit: robot stretch_description, 46 links, 45 joints
Joints:
- joint joint_head_tilt: limit lower=-1.53 upper=0.79 effort=100 velocity=1.0 -> lower=-1.53 upper=0.79 effort=100 velocity=10.0
