Commit message: removed absolute paths from iCub URDF files by replacing them with relative URIs

File: resources/multiverse_episodes/icub_montessori_no_hands/models/iCub.urdf (robot description, URDF)
Before this commit: robot iCub, 105 links, 104 joints
Links:
- link chest: geometry visual mesh filename=file://iCub/meshes/stl/sim_icub3_chest_prt.stl scale=0.0010000000474974513 0.0010000000474974513 0.0010000000474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
- link head: geometry visual mesh filename=file://iCub/meshes/stl/sim_head_head_prt.stl scale=0.0010000000474974513 0.0010000000474974513 0.0010000000474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
- link l_ankle_1: geometry visual mesh filename=file://iCub/meshes/stl/sim_icub3_l_ankle_1_prt.stl scale=0.0010000000474974513 0.0010000000474974513 0.0010000000474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
- link l_ankle_2: geometry visual mesh filename=file://iCub/meshes/stl/sim_icub3_l_ankle_2_prt.stl scale=0.0010000000474974513 0.0010000000474974513 0.0010000000474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
- link l_elbow_1: geometry visual mesh filename=file://iCub/meshes/stl/sim_icub3_l_elbow_1_prt.stl scale=0.0010000000474974513 0.0010000000474974513 0.0010000000474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
- link l_foot_front: geometry visual mesh filename=file://iCub/meshes/stl/sim_icub3_l_foot_front_prt.stl scale=0.0010000000474974513 0.0010000000474974513 0.0010000000474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
- link l_foot_rear: geometry visual mesh filename=file://iCub/meshes/stl/sim_icub3_l_foot_rear_prt.stl scale=0.0010000000474974513 0.0010000000474974513 0.0010000000474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
- link l_forearm: geometry visual mesh filename=file://iCub/meshes/stl/sim_icub3_l_forearm_prt.stl scale=0.0010000000474974513 0.0010000000474974513 0.0010000000474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
- link l_hand: geometry visual mesh filename=file://iCub/meshes/stl/full_LeftHandPalm.stl scale=1.0 1.0 1.0; visual mesh filename=file://iCub/meshes/stl/full_LeftTopCover.stl scale=1.0 1.0 1.0
- link l_hand_index_0: geometry visual mesh filename=file://iCub/meshes/stl/full_LeftIndex0.stl scale=1.0 1.0 1.0
- link l_hand_index_1: geometry visual mesh filename=file://iCub/meshes/stl/full_LeftIndex1.stl scale=1.0 1.0 1.0
- link l_hand_index_2: geometry visual mesh filename=file://iCub/meshes/stl/full_LeftIndex2.stl scale=1.0 1.0 1.0
- link l_hand_index_3: geometry visual mesh filename=file://iCub/meshes/stl/full_LeftIndex3.stl scale=1.0 1.0 1.0
- link l_hand_little_0: geometry visual mesh filename=file://iCub/meshes/stl/full_LeftLittle0.stl scale=1.0 1.0 1.0
- link l_hand_little_1: geometry visual mesh filename=file://iCub/meshes/stl/full_LeftLittle1.stl scale=1.0 1.0 1.0
- link l_hand_little_2: geometry visual mesh filename=file://iCub/meshes/stl/full_LeftLittle2.stl scale=1.0 1.0 1.0
- link l_hand_little_3: geometry visual mesh filename=file://iCub/meshes/stl/full_LeftLittle3.stl scale=1.0 1.0 1.0
- link l_hand_middle_0: geometry visual mesh filename=file://iCub/meshes/stl/full_LeftMiddle0.stl scale=1.0 1.0 1.0
- link l_hand_middle_1: geometry visual mesh filename=file://iCub/meshes/stl/full_LeftMiddle1.stl scale=1.0 1.0 1.0
- link l_hand_middle_2: geometry visual mesh filename=file://iCub/meshes/stl/full_LeftMiddle2.stl scale=1.0 1.0 1.0
- link l_hand_middle_3: geometry visual mesh filename=file://iCub/meshes/stl/full_LeftMiddle3.stl scale=1.0 1.0 1.0
- link l_hand_ring_0: geometry visual mesh filename=file://iCub/meshes/stl/full_LeftRing0.stl scale=1.0 1.0 1.0
- link l_hand_ring_1: geometry visual mesh filename=file://iCub/meshes/stl/full_LeftRing1.stl scale=1.0 1.0 1.0
- link l_hand_ring_2: geometry visual mesh filename=file://iCub/meshes/stl/full_LeftRing2.stl scale=1.0 1.0 1.0
- link l_hand_ring_3: geometry visual mesh filename=file://iCub/meshes/stl/full_LeftRing3.stl scale=1.0 1.0 1.0
- link l_hand_thumb_0: geometry visual mesh filename=file://iCub/meshes/stl/full_LeftThumb0.stl scale=1.0 1.0 1.0
- link l_hand_thumb_1: geometry visual mesh filename=file://iCub/meshes/stl/full_LeftThumb1.stl scale=1.0 1.0 1.0
- link l_hand_thumb_2: geometry visual mesh filename=file://iCub/meshes/stl/full_LeftThumb2.stl scale=1.0 1.0 1.0
- link l_hand_thumb_3: geometry visual mesh filename=file://iCub/meshes/stl/full_LeftThumb3.stl scale=1.0 1.0 1.0
- link l_hip_1: geometry visual mesh filename=file://iCub/meshes/stl/sim_icub3_l_hip_1_prt.stl scale=0.0010000000474974513 0.0010000000474974513 0.0010000000474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
- link l_hip_2: geometry visual mesh filename=file://iCub/meshes/stl/sim_icub3_l_hip_2_prt.stl scale=0.0010000000474974513 0.0010000000474974513 0.0010000000474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
- link l_hip_3: geometry visual mesh filename=file://iCub/meshes/stl/sim_icub3_l_hip_3_prt.stl scale=0.0010000000474974513 0.0010000000474974513 0.0010000000474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
- link l_lower_leg: geometry visual mesh filename=file://iCub/meshes/stl/sim_icub3_l_lower_leg_prt.stl scale=0.0010000000474974513 0.0010000000474974513 0.0010000000474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
- link l_shoulder_1: geometry visual mesh filename=file://iCub/meshes/stl/sim_icub3_l_shoulder_1_prt.stl scale=0.0010000000474974513 0.0010000000474974513 0.0010000000474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
- link l_shoulder_2: geometry visual mesh filename=file://iCub/meshes/stl/sim_icub3_l_shoulder_2_prt.stl scale=0.0010000000474974513 0.0010000000474974513 0.0010000000474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
- link l_shoulder_3: geometry visual mesh filename=file://iCub/meshes/stl/sim_icub3_l_shoulder_3_prt.stl scale=0.0010000000474974513 0.0010000000474974513 0.0010000000474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
- link l_upper_arm: geometry visual mesh filename=file://iCub/meshes/stl/sim_icub3_l_upperarm_prt.stl scale=0.0010000000474974513 0.0010000000474974513 0.0010000000474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
- link l_upper_leg: geometry visual mesh filename=file://iCub/meshes/stl/sim_icub3_l_upper_leg_prt.stl scale=0.0010000000474974513 0.0010000000474974513 0.0010000000474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
- link l_wrist_1: geometry visual mesh filename=file://iCub/meshes/stl/sim_icub3_l_wrist_1_prt.stl scale=0.0010000000474974513 0.0010000000474974513 0.0010000000474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
- link neck_1: geometry visual mesh filename=file://iCub/meshes/stl/sim_head_neck_1_prt.stl scale=0.0010000000474974513 0.0010000000474974513 0.0010000000474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
- link neck_2: geometry visual mesh filename=file://iCub/meshes/stl/sim_head_neck_2_prt.stl scale=0.0010000000474974513 0.0010000000474974513 0.0010000000474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
- link neck_3: geometry visual mesh filename=file://iCub/meshes/stl/sim_head_neck_3_prt.stl scale=0.0010000000474974513 0.0010000000474974513 0.0010000000474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
- link r_ankle_1: geometry visual mesh filename=file://iCub/meshes/stl/sim_icub3_r_ankle_1_prt.stl scale=0.0010000000474974513 0.0010000000474974513 0.0010000000474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
- link r_ankle_2: geometry visual mesh filename=file://iCub/meshes/stl/sim_icub3_r_ankle_2_prt.stl scale=0.0010000000474974513 0.0010000000474974513 0.0010000000474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
- link r_elbow_1: geometry visual mesh filename=file://iCub/meshes/stl/sim_icub3_r_elbow_1_prt.stl scale=0.0010000000474974513 0.0010000000474974513 0.0010000000474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
- link r_foot_front: geometry visual mesh filename=file://iCub/meshes/stl/sim_icub3_r_foot_front_prt.stl scale=0.0010000000474974513 0.0010000000474974513 0.0010000000474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
- link r_foot_rear: geometry visual mesh filename=file://iCub/meshes/stl/sim_icub3_r_foot_rear_prt.stl scale=0.0010000000474974513 0.0010000000474974513 0.0010000000474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
- link r_forearm: geometry visual mesh filename=file://iCub/meshes/stl/sim_icub3_r_forearm_prt.stl scale=0.0010000000474974513 0.0010000000474974513 0.0010000000474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
- link r_hand: geometry visual mesh filename=file://iCub/meshes/stl/full_RightHandPalm.stl scale=1.0 1.0 1.0; visual mesh filename=file://iCub/meshes/stl/full_RightTopCover.stl scale=0.0010000000474974513 0.0010000000474974513 0.0010000000474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
- link r_hand_index_0: geometry visual mesh filename=file://iCub/meshes/stl/full_RightIndex0.stl scale=1.0 1.0 1.0
- link r_hand_index_1: geometry visual mesh filename=file://iCub/meshes/stl/full_RightIndex1.stl scale=1.0 1.0 1.0
- link r_hand_index_2: geometry visual mesh filename=file://iCub/meshes/stl/full_RightIndex2.stl scale=1.0 1.0 1.0
- link r_hand_index_3: geometry visual mesh filename=file://iCub/meshes/stl/full_RightIndex3.stl scale=1.0 1.0 1.0
- link r_hand_little_0: geometry visual mesh filename=file://iCub/meshes/stl/full_RightLittle0.stl scale=1.0 1.0 1.0
- link r_hand_little_1: geometry visual mesh filename=file://iCub/meshes/stl/full_RightLittle1.stl scale=1.0 1.0 1.0
- link r_hand_little_2: geometry visual mesh filename=file://iCub/meshes/stl/full_RightLittle2.stl scale=1.0 1.0 1.0
- link r_hand_little_3: geometry visual mesh filename=file://iCub/meshes/stl/full_RightLittle3.stl scale=1.0 1.0 1.0
- link r_hand_middle_0: geometry visual mesh filename=file://iCub/meshes/stl/full_RightMiddle0.stl scale=1.0 1.0 1.0
- link r_hand_middle_1: geometry visual mesh filename=file://iCub/meshes/stl/full_RightMiddle1.stl scale=1.0 1.0 1.0
- link r_hand_middle_2: geometry visual mesh filename=file://iCub/meshes/stl/full_RightMiddle2.stl scale=1.0 1.0 1.0
- link r_hand_middle_3: geometry visual mesh filename=file://iCub/meshes/stl/full_RightMiddle3.stl scale=1.0 1.0 1.0
- link r_hand_ring_0: geometry visual mesh filename=file://iCub/meshes/stl/full_RightRing0.stl scale=1.0 1.0 1.0
- link r_hand_ring_1: geometry visual mesh filename=file://iCub/meshes/stl/full_RightRing1.stl scale=1.0 1.0 1.0
- link r_hand_ring_2: geometry visual mesh filename=file://iCub/meshes/stl/full_RightRing2.stl scale=1.0 1.0 1.0
- link r_hand_ring_3: geometry visual mesh filename=file://iCub/meshes/stl/full_RightRing3.stl scale=1.0 1.0 1.0
- link r_hand_thumb_0: geometry visual mesh filename=file://iCub/meshes/stl/full_RightThumb0.stl scale=1.0 1.0 1.0
- link r_hand_thumb_1: geometry visual mesh filename=file://iCub/meshes/stl/full_RightThumb1.stl scale=1.0 1.0 1.0
- link r_hand_thumb_2: geometry visual mesh filename=file://iCub/meshes/stl/full_RightThumb2.stl scale=1.0 1.0 1.0
- link r_hand_thumb_3: geometry visual mesh filename=file://iCub/meshes/stl/full_RightThumb3.stl scale=1.0 1.0 1.0
- link r_hip_1: geometry visual mesh filename=file://iCub/meshes/stl/sim_icub3_r_hip_1_prt.stl scale=0.0010000000474974513 0.0010000000474974513 0.0010000000474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
- link r_hip_2: geometry visual mesh filename=file://iCub/meshes/stl/sim_icub3_r_hip_2_prt.stl scale=0.0010000000474974513 0.0010000000474974513 0.0010000000474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
- link r_hip_3: geometry visual mesh filename=file://iCub/meshes/stl/sim_icub3_r_hip_3_prt.stl scale=0.0010000000474974513 0.0010000000474974513 0.0010000000474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
- link r_lower_leg: geometry visual mesh filename=file://iCub/meshes/stl/sim_icub3_r_lower_leg_prt.stl scale=0.0010000000474974513 0.0010000000474974513 0.0010000000474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
- link r_shoulder_1: geometry visual mesh filename=file://iCub/meshes/stl/sim_icub3_r_shoulder_1_prt.stl scale=0.0010000000474974513 0.0010000000474974513 0.0010000000474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
- link r_shoulder_2: geometry visual mesh filename=file://iCub/meshes/stl/sim_icub3_r_shoulder_2_prt.stl scale=0.0010000000474974513 0.0010000000474974513 0.0010000000474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
- link r_shoulder_3: geometry visual mesh filename=file://iCub/meshes/stl/sim_icub3_r_shoulder_3_prt.stl scale=0.0010000000474974513 0.0010000000474974513 0.0010000000474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
- link r_upper_arm: geometry visual mesh filename=file://iCub/meshes/stl/sim_icub3_r_upperarm_prt.stl scale=0.0010000000474974513 0.0010000000474974513 0.0010000000474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
- link r_upper_leg: geometry visual mesh filename=file://iCub/meshes/stl/sim_icub3_r_upper_leg_prt.stl scale=0.0010000000474974513 0.0010000000474974513 0.0010000000474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
- link r_wrist_1: geometry visual mesh filename=file://iCub/meshes/stl/sim_icub3_r_wrist_1_prt.stl scale=0.0010000000474974513 0.0010000000474974513 0.0010000000474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
- link root_link: geometry visual mesh filename=file://iCub/meshes/stl/sim_icub3_root_link_prt.stl scale=0.0010000000474974513 0.0010000000474974513 0.0010000000474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
- link torso_1: geometry visual mesh filename=file://iCub/meshes/stl/sim_icub3_torso_1_prt.stl scale=0.0010000000474974513 0.0010000000474974513 0.0010000000474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
- link torso_2: geometry visual mesh filename=file://iCub/meshes/stl/sim_icub3_torso_2_prt.stl scale=0.0010000000474974513 0.0010000000474974513 0.0010000000474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
