Commit message: [DAiSy] added velocity interface

File: semantic_digital_twin/resources/urdf/daisy.urdf (robot description, URDF)
Before this commit: robot daisy, 40 links, 39 joints
Joints:
- joint left_elbow_joint: origin xyz=-0.4253042110231258 0 0 rpy=0.0004004671080040561 0.0009514770223369379 -1.7924730990257e-05 -> xyz=-0.425 0 0 rpy=0 0 0
- joint left_kms_mounting_plate_joint: parent left_ft_frame -> left_tool0
- joint left_shoulder_lift_joint: origin xyz=0.0003389259895244025 0 0 rpy=1.570188630966205 0 -2.265958458696488e-05 -> xyz=0 0 0 rpy=1.570796327 0 0
- joint left_shoulder_pan_joint: origin xyz=0 0 0.08926862022354863 rpy=0 0 -3.110709810076213e-05 -> xyz=0 0 0.089159 rpy=0 0 0
- joint left_wrist_1_joint: origin xyz=-0.3922027350666989 -0.000205976121060937 0.1110693431741534 rpy=0.001854480084698149 0.002132283504831872 -2.832733147845861e-05 -> xyz=-0.39225 0 0.10915 rpy=0 0 0
- joint left_wrist_2_joint: origin xyz=-1.197491683347993e-05 -0.09487067619053229 2.624213932941136e-05 rpy=1.570519717206836 0 -3.042567573180347e-05 -> xyz=0 -0.09465 -1.941303950897609e-11 rpy=1.570796327 0 0
- joint left_wrist_3_joint: origin xyz=3.793182170272546e-05 0.08257810081734195 4.939571689165691e-06 rpy=1.570856143763734 3.141592653589793 -3.141564220604994 -> xyz=0 0.0823 -1.688001216681175e-11 rpy=1.570796326589793 3.141592653589793 3.141592653589793
- joint right_kms_mounting_plate_joint: parent right_ft_frame -> right_tool0
