Commit message: remove apartment changes

File: pycram/resources/worlds/apartment.urdf (robot description, URDF)
Before this commit: robot apartment, 113 links, 112 joints
Joints:
- joint cabinet2_door_out_joint: mimic (none) -> joint=cabinet2_door_left_joint multiplier=0.01
- joint cabinet3_door_bottom_out_joint: mimic (none) -> joint=cabinet3_door_bottom_left_joint multiplier=0.01
- joint cabinet3_door_top_out_joint: mimic (none) -> joint=cabinet3_door_top_left_joint multiplier=0.01

Commit message: first att

File: pycram/resources/worlds/apartment.urdf (robot description, URDF)
Before this commit: robot apartment, 109 links, 108 joints
Links:
- link cabinet1: geometry collision mesh filename=package://iai_apartment/meshes/cabinet01/IAICabinet1W60.obj; visual mesh filename=package://iai_apartment/meshes/cabinet01/IAICabinet1W60_woo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
- link cabinet1_door_top_left: geometry collision mesh filename=package://iai_apartment/meshes/cabinet01/IAIDoorW60H80.obj; visual mesh filename=package://iai_apartment/meshes/cabinet01/IAIDoorW60H80_wood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
- link cabinet1_drawer_bottom: geometry collision mesh filename=package://iai_apartment/meshes/cabinet01/IAIDrawerW60H53.obj; visual mesh filename=package://iai_apartment/meshes/cabinet01/IAIDrawerW60H53_wo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
- link cabinet1_drawer_middle: geometry collision mesh filename=package://iai_apartment/meshes/cabinet01/IAIDrawerW60H26.obj; visual mesh filename=package://iai_apartment/meshes/cabinet01/IAIDrawerW60H26_wo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
- link cabinet2: geometry collision mesh filename=package://iai_apartment/meshes/cabinet02/IAICabinet2W40H57.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; visual mesh filename=package://iai_apartment/meshes/cabinet02/IAICabinet2W40H57_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
- link cabinet2_door_left: geometry collision mesh filename=package://iai_apartment/meshes/cabinet02/IAIDoorW40H212.obj; visual mesh filename=package://iai_apartment/meshes/cabinet02/IAIDoorW40H212_woo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
- link cabinet2_drawer_big: geometry collision mesh filename=package://iai_apartment/meshes/cabinet02/IAIDrawerW40H22.obj; visual mesh filename=package://iai_apartment/meshes/cabinet02/IAIDrawerW40H22_wo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
- link cabinet2_drawer_small: geometry collision mesh filename=package://iai_apartment/meshes/cabinet02/IAIDrawerW40H10.obj; visual mesh filename=package://iai_apartment/meshes/cabinet02/IAIDrawerW40H10_wo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
- link cabinet3: geometry collision mesh filename=package://iai_apartment/meshes/cabinet03/IAICabinet3W60.obj; visual mesh filename=package://iai_apartment/meshes/cabinet03/IAICabinet3W60_woo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
- link cabinet3_door_bottom_left: geometry collision mesh filename=package://iai_apartment/meshes/cabinet03/IAIDoorW60H80.obj; visual mesh filename=package://iai_apartment/meshes/cabinet03/IAIDoorW60H80_wood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
- link cabinet3_door_top_left: geometry collision mesh filename=package://iai_apartment/meshes/cabinet03/IAIDoorW60H133.obj; visual mesh filename=package://iai_apartment/meshes/cabinet03/IAIDoorW60H133_woo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
- link cabinet4_door_bottom: geometry collision mesh filename=package://iai_apartment/meshes/cabinet04/IAIDoor2W100H40.obj; visual mesh filename=package://iai_apartment/meshes/cabinet04/IAIDoor2W100H40_wo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
- link cabinet4_door_top: geometry collision mesh filename=package://iai_apartment/meshes/cabinet04/IAIDoor1W100H40.obj; visual mesh filename=package://iai_apartment/meshes/cabinet04/IAIDoor1W100H40_wo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
- link cooktop: geometry collision mesh filename=package://iai_apartment/meshes/cooktop/IAIKitchenCookTop.obj; visual mesh filename=package://iai_apartment/meshes/cooktop/IAIKitchenCookTop_st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
- link oven: geometry collision box size=0.58 0.58 0.59; visual mesh filename=package://iai_apartment/meshes/cabinet01/oven_metal.obj
- link sink: geometry collision mesh filename=package://iai_apartment/meshes/sink/IAIKitchenSink.obj; visual mesh filename=package://iai_apartment/meshes/sink/IAIKitchenSink_metal.obj
